Commit message: Updated URDF

File: RVIZ/Scara_Arm.urdf (robot description, URDF)
Before this commit: robot flexible, 16 links, 15 joints
Links:
- removed link box
- removed link gripper_pole
- removed link head
- removed link left_back_wheel
- removed link left_base
- removed link left_front_wheel
- removed link left_gripper
- removed link left_leg
- removed link left_tip
- removed link right_back_wheel
- removed link right_base
- removed link right_front_wheel
- removed link right_gripper
- removed link right_leg
- removed link right_tip
- added link Link1; visual mesh filename=package://Scara-Arm/STL/Link 0.stl
- added link Link2; visual mesh filename=package://Scara-Arm/STL/Link 1.stl
- added link ZAxis; visual mesh filename=package://Scara-Arm/STL/Z-Axis.stl
- link base_link: geometry visual mesh filename=package://Scara-Arm/STL/Bottom.stl
Joints:
- removed joint base_to_left_leg
- removed joint base_to_right_leg
- removed joint gripper_extension
- removed joint head_swivel
- removed joint left_back_wheel_joint
- removed joint left_base_joint
- removed joint left_front_wheel_joint
- removed joint left_gripper_joint
- removed joint left_tip_joint
- removed joint right_back_wheel_joint
- removed joint right_base_joint
- removed joint right_front_wheel_joint
- removed joint right_gripper_joint
- removed joint right_tip_joint
- removed joint tobox
- added joint BaseToZAxis: type prismatic, parent base_link, child Link2, origin xyz=0 -0.06 .159 rpy= 0 0 3.14159, axis 0 0 1, limit lower=0 upper=6 effort=1.0 velocity=1.0
- added joint Link1ToLink2: type revolute, parent Link3, child Link4, origin xyz=-0.17 -0.025 0 rpy= 0 0 0, axis 0 1 0, limit lower=0 upper=6 effort=1.0 velocity=1.0
- added joint ZAxisToLink1: type revolute, parent Link2, child Link3, origin xyz=0.05 0 .01 rpy= 0 0 0, axis 0 1 0, limit lower=0 upper=6 effort=1.0 velocity=1.0
