Commit message: Full Working URDF

File: robotarm/ScaraArm/robot_description.urdf (robot description, URDF)
Before this commit: robot visual, 4 links, 3 joints
Links:
- removed link Link3
- removed link Link4
- added link LeadScrew; visual mesh filename=package://robotarm/ScaraArm/Leadscrew.stl scale=0.01 0.01 0.01
- added link Link1; visual mesh filename=package://robotarm/ScaraArm/Link 0.stl scale=0.01 0.01 0.01
- added link Link1Bottom; visual mesh filename=package://robotarm/ScaraArm/Link Bottom.stl scale=0.01 0.01 0.01
- added link Link1Top; visual mesh filename=package://robotarm/ScaraArm/Link_Top.stl scale=0.01 0.01 0.01
- added link Link2Bottom; visual mesh filename=package://robotarm/ScaraArm/Link Bottom.stl scale=0.01 0.01 0.01
- added link Link2Top; visual mesh filename=package://robotarm/ScaraArm/Link_Top.stl scale=0.01 0.01 0.01
- added link SmoothRodL; visual mesh filename=package://robotarm/ScaraArm/SmoothRods.stl scale=0.01 0.01 0.01
- added link SmoothRodR; visual mesh filename=package://robotarm/ScaraArm/SmoothRods.stl scale=0.01 0.01 0.01
- added link Top; visual mesh filename=package://robotarm/ScaraArm/Top.stl scale=0.01 0.01 0.01
- added link Z-Axis; visual mesh filename=package://robotarm/ScaraArm/Z-Axis.stl scale=0.01 0.01 0.01
- added link bottom; visual mesh filename=package://robotarm/ScaraArm/Bottom.stl scale=0.01 0.01 0.01
- link Link2: geometry visual mesh filename=package://robotarm/ScaraArm/Link 0.stl scale=0.01 0.01 0.01
- link base_link: geometry visual cylinder length=0.01 radius=0.01
Joints:
- removed joint BaseToLink2
- removed joint Link2ToLink3
- removed joint Link3ToLink4
- added joint BaseToBottom: type fixed, parent base_link, child bottom, origin xyz=0 0 0 rpy= 1.57 0 1.57, axis 0 1 0, limit lower=0 upper=6 effort=1.0 velocity=1.0
- added joint Bottom-LeadScrew: type fixed, parent bottom, child LeadScrew, origin xyz=-0.04 0 0 rpy= 0 0 0, axis 0 0 1, limit lower=0 upper=6 effort=1.0 velocity=1.0
- added joint Bottom-SmoothRodL: type fixed, parent bottom, child SmoothRodL, origin xyz=0.37 0.2 0.65 rpy= 0 0 0, axis 0 0 1, limit lower=0 upper=6 effort=1.0 velocity=1.0
- added joint Bottom-SmoothRodR: type fixed, parent bottom, child SmoothRodR, origin xyz=0.37 0.2 -0.65 rpy= 0 0 0, axis 0 0 1, limit lower=0 upper=6 effort=1.0 velocity=1.0
- added joint BottomToZ-Axis: type prismatic, parent bottom, child Z-Axis, origin xyz=0 1 0 rpy= 0 1.57 0, axis 0 1 0, limit lower=0 upper=6 effort=1.0 velocity=1.0
- added joint BottomTop: type fixed, parent bottom, child Top, origin xyz=0 5.1 0 rpy= 0 -1.57 3.14, axis 0 0 1, limit lower=0 upper=6 effort=1.0 velocity=1.0
- added joint Link1-Link2Top: type revolute, parent Link1, child Link2Top, origin xyz=0 0.23 2.74 rpy= 0 0 0, axis 0 1 0, limit lower=0 upper=6 effort=1.0 velocity=1.0
- added joint Link1Top-Link1: type fixed, parent Link1Top, child Link1, origin xyz=0 -0.23 -0.64 rpy= 0 0 0, axis 0 0 1, limit lower=0 upper=6 effort=1.0 velocity=1.0
- added joint Link1Top-Link1Bottom: type fixed, parent Link1Top, child Link1Bottom, origin xyz=0 -0.46 0 rpy= 0 0 0, axis 0 1 0, limit lower=0 upper=6 effort=1.0 velocity=1.0
- added joint Link2Top-Link2: type fixed, parent Link2Top, child Link2, origin xyz=0 -0.23 -0.64 rpy= 0 0 0, axis 0 0 1, limit lower=0 upper=6 effort=1.0 velocity=1.0
- added joint Link2Top-Link2Bottom: type fixed, parent Link2Top, child Link2Bottom, origin xyz=0 -0.46 0 rpy= 0 0 0, axis 0 1 0, limit lower=0 upper=6 effort=1.0 velocity=1.0
- added joint Z-Axis-Link1Top: type revolute, parent Z-Axis, child Link1Top, origin xyz=0 0.23 0.64 rpy= 0 0 0, axis 0 1 0, limit lower=0 upper=6 effort=1.0 velocity=1.0
